Commit message: major refactor on comms arch

File: snakesim/resource/snake_robot.urdf (robot description, URDF)
Before this commit: robot SnakeRobot, 8 links, 7 joints
Links:
- removed link base_link
- removed link solid
- removed link solid_0
- removed link solid_1
- removed link solid_2
- removed link solid_3
- removed link solid_4
- removed link solid_5
- added link endEffector
- added link link0; visual box size=0.0451 0.0247 0.034
- added link link1; visual box size=0.01 0.042 0.046; visual box size=0.022 0.02 0.007
- added link link2; visual box size=0.01 0.042 0.046; visual box size=0.022 0.02 0.007
- added link link3; visual box size=0.01 0.042 0.046; visual box size=0.022 0.02 0.007
- added link link4; visual box size=0.01 0.042 0.046; visual box size=0.022 0.02 0.007
- added link link5; visual box size=0.01 0.042 0.046; visual box size=0.022 0.02 0.007
Joints:
- removed joint rotationalMotor6
- removed joint rotationalMotor7
- added joint endEffFrame: type fixed, parent link5, child endEffector, origin xyz=0.02 0 0 rpy=0 0 0, axis 0 0 1
- joint rotationalMotor1: axis 0 1 -0.000004 -> 0 0 1; child solid -> link1; limit effort=10 velocity=10 -> lower=-2.0943 upper=2.0943 effort=10 velocity=10; origin xyz=0 0 0 rpy=1.5708 0 0 -> xyz=0 0 0.0127 rpy=0 -1.5707 0; parent base_link -> link0
- joint rotationalMotor2: axis 0 -1 0.000001 -> 0 0 1; child solid_0 -> link2; limit effort=10 velocity=10 -> lower=-2.0943 upper=2.0943 effort=10 velocity=10; origin xyz=0.06 0 0 rpy=-1.570795 0 0 -> xyz=0.06 0 0 rpy=1.5707 0 0; parent solid -> link1
- joint rotationalMotor3: axis 0 1 -0.000004 -> 0 0 1; child solid_1 -> link3; limit effort=10 velocity=10 -> lower=-2.0943 upper=2.0943 effort=10 velocity=10; origin xyz=0.06 0 0 rpy=1.5708 0 0 -> xyz=0.06 0 0 rpy=-1.5707 0 0; parent solid_0 -> link2
- joint rotationalMotor4: axis 0 -1 0.000001 -> 0 0 1; child solid_2 -> link4; limit effort=10 velocity=10 -> lower=-2.0943 upper=2.0943 effort=10 velocity=10; origin xyz=0.06 0 0 rpy=-1.570795 0 0 -> xyz=0.06 0 0 rpy=1.5707 0 0; parent solid_1 -> link3
- joint rotationalMotor5: axis 0 1 -0.000004 -> 0 0 1; child solid_3 -> link5; limit effort=10 velocity=10 -> lower=-2.0943 upper=2.0943 effort=10 velocity=10; origin xyz=0.06 0 0 rpy=1.5708 0 0 -> xyz=0.06 0 0 rpy=-1.5707 0 0; parent solid_2 -> link4
